File: kicad/C64-Composite-Modulator.kicad_sch (KiCad schematic)
At the start: 48 parts, among them Q1 BC847C, Q2 BC847C, U1 78L05G-AB3-R

Commit message: Reduce the number of JLCPCB's extended parts
Parts:
- C2: LCSC C159777 -> C1739; Manufacturer Samsung Electro-Mechanics -> FH(Guangdong Fenghua Advanced Tech); Mfr.Part CL21B333KBANNNC -> 0805B333K500NT
- L1: LCSC C95978 -> C1046; Mfr.Part MCL2012H100MT -> SDFL2012S100KTF
Changed lines of the file:
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@@
       (effects (font (size 1.27 1.27)) hide)
     )
-    (property "Datasheet" "https://datasheet.lcsc.com/lcsc/1810241123_Samsung-Electro-Mechanics-CL21B333KBANNNC_C159777.pdf" (id 3) (at 85.09 121.92 0)
+    (property "Datasheet" "https://datasheet.lcsc.com/lcsc/1811061723_FH-Guangdong-Fenghua-Advanced-Tech-0805B333K500NT_C1739.pdf" (id 3) (at 85.09 121.92 0)
       (effects (font (size 1.27 1.27)) hide)
     )
@@
       (effects (font (size 1.27 1.27)) hide)
     )
-    (property "Manufacturer" "Samsung Electro-Mechanics" (id 5) (at 85.09 121.92 0)
-      (effects (font (size 1.27 1.27)) hide)
-    )
-    (property "Mfr.Part" "CL21B333KBANNNC" (id 6) (at 85.09 121.92 0)
-      (effects (font (size 1.27 1.27)) hide)
-    )
-    (property "LCSC" "C159777" (id 7) (at 85.09 121.92 0)
+    (property "Manufacturer" "FH(Guangdong Fenghua Advanced Tech)" (id 5) (at 85.09 121.92 0)
+      (effects (font (size 1.27 1.27)) hide)
+    )
+    (property "Mfr.Part" "0805B333K500NT" (id 6) (at 85.09 121.92 0)
+      (effects (font (size 1.27 1.27)) hide)
+    )
+    (property "LCSC" "C1739" (id 7) (at 85.09 121.92 0)
       (effects (font (size 1.27 1.27)) hide)
     )
@@
       (effects (font (size 1.27 1.27)) hide)
     )
-    (property "Datasheet" "https://datasheet.lcsc.com/lcsc/2110081230_Sunlord-MCL2012H100MT_C95978.pdf" (id 3) (at 168.91 93.345 0)
-      (effects (font (size 1.27 1.27)) hide)
-    )
-    (property "Description" "100mA 10uH ±20% 650mΩ 0805 Inductors (SMD) ROHS" (id 4) (at 168.91 93.345 0)
+    (property "Datasheet" "https://datasheet.lcsc.com/lcsc/2110081230_Sunlord-SDFL2012S100KTF_C1046.pdf" (id 3) (at 168.91 93.345 0)
+      (effects (font (size 1.27 1.27)) hide)
+    )
+    (property "Description" "15mA 10uH ±10% 1.15Ω 0805 Inductors (SMD) ROHS" (id 4) (at 168.91 93.345 0)
       (effects (font (size 1.27 1.27)) hide)
     )
@@
       (effects (font (size 1.27 1.27)) hide)
     )
-    (property "Mfr.Part" "MCL2012H100MT" (id 6) (at 168.91 93.345 0)
-      (effects (font (size 1.27 1.27)) hide)
-    )
-    (property "LCSC" "C95978" (id 7) (at 168.91 93.345 0)
-      (effects (font (size 1.27 1.27)) hide)
-    )
+    (property "Mfr.Part" "SDFL2012S100KTF" (id 6) (at 168.91 93.345 0)
+      (effects (font (size 1.27 1.27)) hide)
+    )
+    (property "LCSC" "C1046" (id 7) (at 168.91 93.345 0)
+      (effects (font (size 1.27 1.27)) hide)
+    )
